File: PCB/southpawpcb.kicad_pcb (KiCad board)
At the start: 2 copper layers, 362.9 x 103.6 mm, 162 parts, among them K1 KEYSW, K10 KEYSW, K11 KEYSW, K12 KEYSW, K13 KEYSW, K14 KEYSW, K15 KEYSW, K16 KEYSW, K17 KEYSW, K18 KEYSW, K19 KEYSW, K2 KEYSW, K20 KEYSW, K21 KEYSW, K22 KEYSW, K23 KEYSW, K24 KEYSW, K25 KEYSW, K26 KEYSW, K27 KEYSW, K28 KEYSW, K29 KEYSW, K3 KEYSW, K30 KEYSW, K31 KEYSW, K32 KEYSW, K33 KEYSW, K34 KEYSW, K35 KEYSW, K36 KEYSW, K37 KEYSW, K38 KEYSW, K39 KEYSW, K4 KEYSW, K40 KEYSW, K41 KEYSW, K42 KEYSW, K43 KEYSW, K44 KEYSW, K45 KEYSW, K46 KEYSW, K47 KEYSW, K48 KEYSW, K49 KEYSW, K5 KEYSW, K50 KEYSW, K51 KEYSW, K52 KEYSW, K53 KEYSW, K54 KEYSW, K55 KEYSW, K56 KEYSW, K57 KEYSW, K58 KEYSW, K59 KEYSW, K6 KEYSW, K60 KEYSW, K61 KEYSW, K62 KEYSW, K63 KEYSW, K64 KEYSW, K65 KEYSW, K66 KEYSW, K67 KEYSW, K68 KEYSW, K69 KEYSW, K7 KEYSW, K70 KEYSW, K71 KEYSW, K72 KEYSW, K73 KEYSW, K74 KEYSW, K75 KEYSW, K76 KEYSW, K77 KEYSW, K78 KEYSW, K8 KEYSW, K9 KEYSW, SW1 Reset, U1 ProMicro

Commit message: attempt at retracing
Parts:
- K1, K10, K11, K12, K13, K14, K15, K16, K17, K19, K2, K20, K21, K24, K25, K26, K27, K28, K29, K3, K30, K31, K32, K33, K34, K35, K37, K38, K39, K4, K41, K42, K43, K44, K45, K46, K47, K48, K49, K5, K50, K51, K53, K54, K55, K58, K59, K6, K60, K61, K62, K63, K64, K65, K66, K67, K7, K70, K8, K9: footprint MX/Alps_Hybrid:MX-1U-NoLED -> MX_Only:MXOnly-1U-Hotswap
- K18, K22, K56, K69: footprint MX/Alps_Hybrid:MX-2U-NoLED -> MX_Only:MXOnly-2U-Hotswap
- K23, K36: footprint MX/Alps_Hybrid:MX-1.5U-NoLED -> MX_Only:MXOnly-1.5U-Hotswap
- K40: footprint MX/Alps_Hybrid:MX-1.75U-NoLED -> MX_Only:MXOnly-1.75U-Hotswap
- K52, K57: footprint MX/Alps_Hybrid:MX-2.25U-NoLED -> MX_Only:MXOnly-2.25U-Hotswap
- K68: footprint MX/Alps_Hybrid:MX-2.75U-NoLED -> MX_Only:MXOnly-2.75U-Hotswap
- K71, K72, K73, K75, K76, K77, K78: footprint MX/Alps_Hybrid:MX-1.25U-NoLED -> MX_Only:MXOnly-1.25U-Hotswap
- K74: footprint MX/Alps_Hybrid:MX-6.25U-NoLED -> MX_Only:MXOnly-6.25U-Hotswap
- U1: footprint Pro_Micro:ProMicro -> promicro:ProMicro
- moved U1 0.22 mm to (43.2, -9.49)
- turned K2 to 270 degrees
- turned K20 to 270 degrees
Connections:
- K1 pad 2: Net-(D1-Pad2) -> Net-(K1-Pad2)
- K10 pad 1: Net-(K1-Pad1) -> Net-(K10-Pad1)
- K10 pad 2: Net-(D10-Pad2) -> Net-(K10-Pad2)
- K11 pad 2: Net-(D11-Pad2) -> Net-(K11-Pad2)
- K12 pad 2: Net-(D12-Pad2) -> Net-(K12-Pad2)
- K13 pad 2: Net-(D13-Pad2) -> Net-(K13-Pad2)
- K14 pad 2: Net-(D14-Pad2) -> Net-(K14-Pad2)
- K15 pad 2: Net-(D15-Pad2) -> Net-(K15-Pad2)
- K16 pad 2: Net-(D16-Pad2) -> Net-(K16-Pad2)
- K17 pad 2: Net-(D17-Pad2) -> Net-(K17-Pad2)
- K18 pad 2: Net-(D18-Pad2) -> Net-(K18-Pad2)
- K19 pad 1: Net-(K1-Pad1) -> Net-(K19-Pad1)
- K19 pad 2: Net-(D19-Pad2) -> Net-(K19-Pad2)
- K2 pad 1: Net-(K11-Pad1) -> Net-(K2-Pad1)
- K2 pad 2: Net-(D2-Pad2) -> Net-(U1-Pad20)
- K20 pad 1: Net-(K11-Pad1) -> Net-(K20-Pad1)
- K20 pad 2: Net-(D20-Pad2) -> Net-(U1-Pad20)
- K21 pad 1: Net-(K12-Pad1) -> Net-(K21-Pad1)
- K21 pad 2: Net-(D21-Pad2) -> Net-(K21-Pad2)
- K22 pad 1: Net-(K13-Pad1) -> Net-(K22-Pad1)
- K22 pad 2: Net-(D22-Pad2) -> Net-(K22-Pad2)
- K23 pad 1: Net-(K14-Pad1) -> Net-(K23-Pad1)
- K23 pad 2: Net-(D23-Pad2) -> Net-(K23-Pad2)
- K24 pad 1: Net-(K15-Pad1) -> Net-(K24-Pad1)
- K24 pad 2: Net-(D24-Pad2) -> Net-(K24-Pad2)
- K25 pad 1: Net-(K16-Pad1) -> Net-(K25-Pad1)
- K25 pad 2: Net-(D25-Pad2) -> Net-(K25-Pad2)
- K26 pad 1: Net-(K17-Pad1) -> Net-(K26-Pad1)
- K26 pad 2: Net-(D26-Pad2) -> Net-(K26-Pad2)
- K27 pad 1: Net-(K18-Pad1) -> Net-(K27-Pad1)
- K27 pad 2: Net-(D27-Pad2) -> Net-(K27-Pad2)
- K28 pad 1: Net-(K1-Pad1) -> Net-(K28-Pad1)
- K28 pad 2: Net-(D28-Pad2) -> Net-(K28-Pad2)
- K29 pad 1: Net-(K11-Pad1) -> Net-(K29-Pad1)
- K29 pad 2: Net-(D29-Pad2) -> Net-(K29-Pad2)
- K3 pad 1: Net-(K12-Pad1) -> Net-(K3-Pad1)
- K3 pad 2: Net-(D3-Pad2) -> Net-(K3-Pad2)
- K30 pad 1: Net-(K12-Pad1) -> Net-(K30-Pad1)
- K30 pad 2: Net-(D30-Pad2) -> Net-(K30-Pad2)
- K31 pad 1: Net-(K13-Pad1) -> Net-(K31-Pad1)
- K31 pad 2: Net-(D31-Pad2) -> Net-(K31-Pad2)
- K32 pad 1: Net-(K14-Pad1) -> Net-(K32-Pad1)
- K32 pad 2: Net-(D32-Pad2) -> Net-(K32-Pad2)
- K33 pad 1: Net-(K15-Pad1) -> Net-(K33-Pad1)
- K33 pad 2: Net-(D33-Pad2) -> Net-(K33-Pad2)
- K34 pad 1: Net-(K16-Pad1) -> Net-(K34-Pad1)
- K34 pad 2: Net-(D34-Pad2) -> Net-(K34-Pad2)
- K35 pad 1: Net-(K17-Pad1) -> Net-(K35-Pad1)
- K35 pad 2: Net-(D35-Pad2) -> Net-(K35-Pad2)
- K36 pad 1: Net-(K18-Pad1) -> Net-(K36-Pad1)
- K36 pad 2: Net-(D36-Pad2) -> Net-(K36-Pad2)
- K37 pad 1: Net-(K1-Pad1) -> Net-(K37-Pad1)
- K37 pad 2: Net-(D37-Pad2) -> Net-(K37-Pad2)
- K38 pad 1: Net-(K11-Pad1) -> Net-(K38-Pad1)
- K38 pad 2: Net-(D38-Pad2) -> Net-(K38-Pad2)
- K39 pad 1: Net-(K12-Pad1) -> Net-(K39-Pad1)
- K39 pad 2: Net-(D39-Pad2) -> Net-(K39-Pad2)
- K4 pad : (no net) -> Net-(U1-Pad18)
- K4 pad 1: Net-(K13-Pad1) -> Net-(K4-Pad1)
- K4 pad 2: Net-(D4-Pad2) -> Net-(K4-Pad2)
- K40 pad 1: Net-(K13-Pad1) -> Net-(K40-Pad1)
- K40 pad 2: Net-(D40-Pad2) -> Net-(K40-Pad2)
- K41 pad 1: Net-(K14-Pad1) -> Net-(K41-Pad1)
- K41 pad 2: Net-(D41-Pad2) -> Net-(K41-Pad2)
- K42 pad 1: Net-(K15-Pad1) -> Net-(K42-Pad1)
- K42 pad 2: Net-(D42-Pad2) -> Net-(K42-Pad2)
- K43 pad 1: Net-(K16-Pad1) -> Net-(K43-Pad1)
- K43 pad 2: Net-(D43-Pad2) -> Net-(K43-Pad2)
- K44 pad 1: Net-(K17-Pad1) -> Net-(K44-Pad1)
- K44 pad 2: Net-(D44-Pad2) -> Net-(K44-Pad2)
- K45 pad 1: Net-(K18-Pad1) -> Net-(K45-Pad1)
- K45 pad 2: Net-(D45-Pad2) -> Net-(K45-Pad2)
- K46 pad 1: Net-(K1-Pad1) -> Net-(K46-Pad1)
- K46 pad 2: Net-(D46-Pad2) -> Net-(K46-Pad2)
- K47 pad 1: Net-(K11-Pad1) -> Net-(K47-Pad1)
- K47 pad 2: Net-(D47-Pad2) -> Net-(K47-Pad2)
- K48 pad 1: Net-(K12-Pad1) -> Net-(K48-Pad1)
- K48 pad 2: Net-(D48-Pad2) -> Net-(K48-Pad2)
- K49 pad 1: Net-(K13-Pad1) -> Net-(K49-Pad1)
- K49 pad 2: Net-(D49-Pad2) -> Net-(K49-Pad2)
- K5 pad 1: Net-(K14-Pad1) -> Net-(K5-Pad1)
- K5 pad 2: Net-(D5-Pad2) -> Net-(K5-Pad2)
- K50 pad 1: Net-(K14-Pad1) -> Net-(K50-Pad1)
- K50 pad 2: Net-(D50-Pad2) -> Net-(K50-Pad2)
- K51 pad 1: Net-(K15-Pad1) -> Net-(K51-Pad1)
- K51 pad 2: Net-(D51-Pad2) -> Net-(K51-Pad2)
- K52 pad 1: Net-(K16-Pad1) -> Net-(K52-Pad1)
- K52 pad 2: Net-(D52-Pad2) -> Net-(K52-Pad2)
- K53 pad 1: Net-(K17-Pad1) -> Net-(K53-Pad1)
- K53 pad 2: Net-(D53-Pad2) -> Net-(K53-Pad2)
- K54 pad 1: Net-(K18-Pad1) -> Net-(K54-Pad1)
- K54 pad 2: Net-(D54-Pad2) -> Net-(K54-Pad2)
- K55 pad 1: Net-(K1-Pad1) -> Net-(K55-Pad1)
- K55 pad 2: Net-(D55-Pad2) -> Net-(K55-Pad2)
- K56 pad 1: Net-(K11-Pad1) -> Net-(K56-Pad1)
- K56 pad 2: Net-(D56-Pad2) -> Net-(K56-Pad2)
- K57 pad 1: Net-(K12-Pad1) -> Net-(K57-Pad1)
- K57 pad 2: Net-(D57-Pad2) -> Net-(K57-Pad2)
- K58 pad 1: Net-(K13-Pad1) -> Net-(K58-Pad1)
- K58 pad 2: Net-(D58-Pad2) -> Net-(K58-Pad2)
- K59 pad 1: Net-(K14-Pad1) -> Net-(K59-Pad1)
- K59 pad 2: Net-(D59-Pad2) -> Net-(K59-Pad2)
- K6 pad : (no net) -> Net-(U1-Pad16)
- K6 pad 1: Net-(K15-Pad1) -> Net-(K6-Pad1)
- K6 pad 2: Net-(D6-Pad2) -> Net-(K6-Pad2)
- K60 pad 1: Net-(K15-Pad1) -> Net-(K60-Pad1)
- K60 pad 2: Net-(D60-Pad2) -> Net-(K60-Pad2)
- K61 pad 1: Net-(K16-Pad1) -> Net-(K61-Pad1)
- K61 pad 2: Net-(D61-Pad2) -> Net-(K61-Pad2)
- K62 pad 1: Net-(K17-Pad1) -> Net-(K62-Pad1)
- K62 pad 2: Net-(D62-Pad2) -> Net-(K62-Pad2)
- K63 pad 1: Net-(K18-Pad1) -> Net-(K63-Pad1)
- K63 pad 2: Net-(D63-Pad2) -> Net-(K63-Pad2)
- K64 pad 1: Net-(K1-Pad1) -> Net-(K64-Pad1)
- K64 pad 2: Net-(D64-Pad2) -> Net-(K64-Pad2)
- K65 pad 1: Net-(K11-Pad1) -> Net-(K65-Pad1)
- K65 pad 2: Net-(D65-Pad2) -> Net-(K65-Pad2)
- K66 pad 1: Net-(K12-Pad1) -> Net-(K66-Pad1)
- K66 pad 2: Net-(D66-Pad2) -> Net-(K66-Pad2)
- K67 pad 1: Net-(K13-Pad1) -> Net-(K67-Pad1)
- K67 pad 2: Net-(D67-Pad2) -> Net-(K67-Pad2)
- K68 pad 1: Net-(K14-Pad1) -> Net-(K68-Pad1)
- K68 pad 2: Net-(D68-Pad2) -> Net-(K68-Pad2)
- K69 pad 1: Net-(K15-Pad1) -> Net-(K69-Pad1)
- K69 pad 2: Net-(D69-Pad2) -> Net-(K69-Pad2)
- K7 pad 1: Net-(K16-Pad1) -> Net-(K7-Pad1)
- K7 pad 2: Net-(D7-Pad2) -> Net-(K7-Pad2)
- K70 pad 1: Net-(K16-Pad1) -> Net-(K70-Pad1)
- K70 pad 2: Net-(D70-Pad2) -> Net-(K70-Pad2)
- K71 pad 1: Net-(K17-Pad1) -> Net-(K71-Pad1)
- K71 pad 2: Net-(D71-Pad2) -> Net-(K71-Pad2)
- K72 pad 1: Net-(K18-Pad1) -> Net-(K72-Pad1)
- K72 pad 2: Net-(D72-Pad2) -> Net-(K72-Pad2)
- K73 pad 1: Net-(K1-Pad1) -> Net-(K73-Pad1)
- K73 pad 2: Net-(D73-Pad2) -> Net-(K73-Pad2)
- K74 pad 1: Net-(K11-Pad1) -> Net-(K74-Pad1)
- K74 pad 2: Net-(D74-Pad2) -> Net-(K74-Pad2)
- K75 pad 1: Net-(K12-Pad1) -> Net-(K75-Pad1)
- K75 pad 2: Net-(D75-Pad2) -> Net-(K75-Pad2)
- K76 pad 1: Net-(K13-Pad1) -> Net-(K76-Pad1)
- K76 pad 2: Net-(D76-Pad2) -> Net-(K76-Pad2)
- K77 pad 1: Net-(K14-Pad1) -> Net-(K77-Pad1)
- K77 pad 2: Net-(D77-Pad2) -> Net-(K77-Pad2)
- K78 pad 1: Net-(K15-Pad1) -> Net-(K78-Pad1)
- K78 pad 2: Net-(D78-Pad2) -> Net-(K78-Pad2)
- K8 pad 1: Net-(K17-Pad1) -> Net-(K8-Pad1)
- K8 pad 2: Net-(D8-Pad2) -> Net-(K8-Pad2)
- K9 pad 1: Net-(K18-Pad1) -> Net-(K9-Pad1)
- K9 pad 2: Net-(D9-Pad2) -> Net-(K9-Pad2)
- U1 pad 12: Net-(K1-Pad1) -> Net-(U1-Pad12)
- U1 pad 13: Net-(K18-Pad1) -> Net-(U1-Pad13)
- U1 pad 14: Net-(K17-Pad1) -> Net-(U1-Pad14)
- U1 pad 15: Net-(K16-Pad1) -> Net-(U1-Pad15)
- U1 pad 16: Net-(K15-Pad1) -> Net-(U1-Pad16)
- U1 pad 17: Net-(K14-Pad1) -> Net-(U1-Pad17)
- U1 pad 18: Net-(K13-Pad1) -> Net-(U1-Pad18)
- U1 pad 19: Net-(K12-Pad1) -> Net-(U1-Pad19)
- U1 pad 20: Net-(K11-Pad1) -> Net-(U1-Pad20)
- U1 pad 22: Net-(SW1-Pad2) -> Net-(U1-Pad22)
- U1 pad 23: Net-(SW1-Pad1) -> Net-(U1-Pad23)
Routing:
- net (no net): track 0.00 -> 1599.0 mm
- net Net-(K18-Pad1): track 523.6 -> 2.00 mm
- net Net-(K17-Pad1): track 536.8 -> 24.9 mm
- net Net-(K73-Pad1): track 0.00 -> 431.4 mm
- net Net-(K15-Pad1): track 537.3 -> 187.0 mm
- net Net-(K11-Pad1): track 416.4 -> 67.8 mm
- net Net-(K12-Pad1): track 431.4 -> 137.4 mm
- net Net-(K13-Pad1): track 416.2 -> 229.7 mm
- net Net-(U1-Pad16): track 0.00 -> 167.1 mm
- net Net-(K16-Pad1): track 510.4 -> 354.7 mm
- net Net-(K14-Pad1): track 452.0 -> 301.4 mm
- net Net-(K65-Pad1): track 0.00 -> 125.9 mm
- net Net-(K1-Pad1): track 418.1 -> 319.9 mm
- net Net-(K48-Pad1): track 0.00 -> 65.9 mm
- net Net-(U1-Pad20): track 0.00 -> 63.9 mm
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
Commit message: all routed
Parts:
- removed G***: LOGO, Logos:designedbykelvinhallcopy
- removed G***: LOGO, Logos:designedbykelvinhall
- removed G***: LOGO, Logos:southpaw75smallcopy
- removed G***: LOGO, Logos:southpaw75small
- turned K3 to 180 degrees
- turned K4 to 180 degrees
Connections:
- K1 pad 2: Net-(K1-Pad2) -> Net-(D1-Pad2)
- K10 pad 1: Net-(K10-Pad1) -> Net-(K1-Pad1)
- K10 pad 2: Net-(K10-Pad2) -> Net-(D10-Pad2)
- K11 pad 2: Net-(K11-Pad2) -> Net-(D11-Pad2)
- K12 pad 2: Net-(K12-Pad2) -> Net-(D12-Pad2)
- K13 pad 2: Net-(K13-Pad2) -> Net-(D13-Pad2)
- K14 pad 2: Net-(K14-Pad2) -> Net-(D14-Pad2)
- K15 pad 2: Net-(K15-Pad2) -> Net-(D15-Pad2)
- K16 pad 2: Net-(K16-Pad2) -> Net-(D16-Pad2)
- K17 pad 2: Net-(K17-Pad2) -> Net-(D17-Pad2)
- K18 pad 2: Net-(K18-Pad2) -> Net-(D18-Pad2)
- K19 pad 1: Net-(K19-Pad1) -> Net-(K1-Pad1)
- K19 pad 2: Net-(K19-Pad2) -> Net-(D19-Pad2)
- K2 pad 1: Net-(K2-Pad1) -> Net-(D2-Pad2)
- K2 pad 2: Net-(U1-Pad20) -> Net-(K11-Pad1)
- K20 pad 1: Net-(K20-Pad1) -> Net-(D20-Pad2)
- K20 pad 2: Net-(U1-Pad20) -> Net-(K11-Pad1)
- K21 pad 1: Net-(K21-Pad1) -> Net-(K12-Pad1)
- K21 pad 2: Net-(K21-Pad2) -> Net-(D21-Pad2)
- K22 pad 1: Net-(K22-Pad1) -> Net-(K13-Pad1)
- K22 pad 2: Net-(K22-Pad2) -> Net-(D22-Pad2)
- K23 pad 1: Net-(K23-Pad1) -> Net-(K14-Pad1)
- K23 pad 2: Net-(K23-Pad2) -> Net-(D23-Pad2)
- K24 pad 1: Net-(K24-Pad1) -> Net-(K15-Pad1)
- K24 pad 2: Net-(K24-Pad2) -> Net-(D24-Pad2)
- K25 pad 1: Net-(K25-Pad1) -> Net-(K16-Pad1)
- K25 pad 2: Net-(K25-Pad2) -> Net-(D25-Pad2)
- K26 pad 1: Net-(K26-Pad1) -> Net-(K17-Pad1)
- K26 pad 2: Net-(K26-Pad2) -> Net-(D26-Pad2)
- K27 pad 1: Net-(K27-Pad1) -> Net-(K18-Pad1)
- K27 pad 2: Net-(K27-Pad2) -> Net-(D27-Pad2)
- K28 pad 1: Net-(K28-Pad1) -> Net-(K1-Pad1)
- K28 pad 2: Net-(K28-Pad2) -> Net-(D28-Pad2)
- K29 pad 1: Net-(K29-Pad1) -> Net-(K11-Pad1)
- K29 pad 2: Net-(K29-Pad2) -> Net-(D29-Pad2)
- K3 pad 1: Net-(K3-Pad1) -> Net-(D3-Pad2)
- K3 pad 2: Net-(K3-Pad2) -> Net-(K12-Pad1)
- K30 pad 1: Net-(K30-Pad1) -> Net-(K12-Pad1)
- K30 pad 2: Net-(K30-Pad2) -> Net-(D30-Pad2)
- K31 pad 1: Net-(K31-Pad1) -> Net-(K13-Pad1)
- K31 pad 2: Net-(K31-Pad2) -> Net-(D31-Pad2)
- K32 pad 1: Net-(K32-Pad1) -> Net-(K14-Pad1)
- K32 pad 2: Net-(K32-Pad2) -> Net-(D32-Pad2)
- K33 pad 1: Net-(K33-Pad1) -> Net-(K15-Pad1)
- K33 pad 2: Net-(K33-Pad2) -> Net-(D33-Pad2)
- K34 pad 1: Net-(K34-Pad1) -> Net-(K16-Pad1)
- K34 pad 2: Net-(K34-Pad2) -> Net-(D34-Pad2)
- K35 pad 1: Net-(K35-Pad1) -> Net-(K17-Pad1)
- K35 pad 2: Net-(K35-Pad2) -> Net-(D35-Pad2)
- K36 pad 1: Net-(K36-Pad1) -> Net-(K18-Pad1)
- K36 pad 2: Net-(K36-Pad2) -> Net-(D36-Pad2)
- K37 pad 1: Net-(K37-Pad1) -> Net-(K1-Pad1)
- K37 pad 2: Net-(K37-Pad2) -> Net-(D37-Pad2)
- K38 pad 1: Net-(K38-Pad1) -> Net-(K11-Pad1)
- K38 pad 2: Net-(K38-Pad2) -> Net-(D38-Pad2)
- K39 pad 1: Net-(K39-Pad1) -> Net-(K12-Pad1)
- K39 pad 2: Net-(K39-Pad2) -> Net-(D39-Pad2)
- K4 pad : Net-(U1-Pad18) -> (no net)
- K4 pad 1: Net-(K4-Pad1) -> Net-(D4-Pad2)
- K4 pad 2: Net-(K4-Pad2) -> Net-(K13-Pad1)
- K40 pad 1: Net-(K40-Pad1) -> Net-(K13-Pad1)
- K40 pad 2: Net-(K40-Pad2) -> Net-(D40-Pad2)
- K41 pad 1: Net-(K41-Pad1) -> Net-(K14-Pad1)
- K41 pad 2: Net-(K41-Pad2) -> Net-(D41-Pad2)
- K42 pad 1: Net-(K42-Pad1) -> Net-(K15-Pad1)
- K42 pad 2: Net-(K42-Pad2) -> Net-(D42-Pad2)
- K43 pad 1: Net-(K43-Pad1) -> Net-(K16-Pad1)
- K43 pad 2: Net-(K43-Pad2) -> Net-(D43-Pad2)
- K44 pad 1: Net-(K44-Pad1) -> Net-(K17-Pad1)
- K44 pad 2: Net-(K44-Pad2) -> Net-(D44-Pad2)
- K45 pad 1: Net-(K45-Pad1) -> Net-(K18-Pad1)
- K45 pad 2: Net-(K45-Pad2) -> Net-(D45-Pad2)
- K46 pad 1: Net-(K46-Pad1) -> Net-(K1-Pad1)
- K46 pad 2: Net-(K46-Pad2) -> Net-(D46-Pad2)
- K47 pad 1: Net-(K47-Pad1) -> Net-(K11-Pad1)
- K47 pad 2: Net-(K47-Pad2) -> Net-(D47-Pad2)
- K48 pad 1: Net-(K48-Pad1) -> Net-(K12-Pad1)
- K48 pad 2: Net-(K48-Pad2) -> Net-(D48-Pad2)
- K49 pad 1: Net-(K49-Pad1) -> Net-(K13-Pad1)
- K49 pad 2: Net-(K49-Pad2) -> Net-(D49-Pad2)
- K5 pad 1: Net-(K5-Pad1) -> Net-(K14-Pad1)
- K5 pad 2: Net-(K5-Pad2) -> Net-(D5-Pad2)
- K50 pad 1: Net-(K50-Pad1) -> Net-(K14-Pad1)
- K50 pad 2: Net-(K50-Pad2) -> Net-(D50-Pad2)
- K51 pad 1: Net-(K51-Pad1) -> Net-(K15-Pad1)
- K51 pad 2: Net-(K51-Pad2) -> Net-(D51-Pad2)
- K52 pad 1: Net-(K52-Pad1) -> Net-(K16-Pad1)
- K52 pad 2: Net-(K52-Pad2) -> Net-(D52-Pad2)
- K53 pad 1: Net-(K53-Pad1) -> Net-(K17-Pad1)
- K53 pad 2: Net-(K53-Pad2) -> Net-(D53-Pad2)
- K54 pad 1: Net-(K54-Pad1) -> Net-(K18-Pad1)
- K54 pad 2: Net-(K54-Pad2) -> Net-(D54-Pad2)
- K55 pad 1: Net-(K55-Pad1) -> Net-(K1-Pad1)
- K55 pad 2: Net-(K55-Pad2) -> Net-(D55-Pad2)
- K56 pad 1: Net-(K56-Pad1) -> Net-(K11-Pad1)
- K56 pad 2: Net-(K56-Pad2) -> Net-(D56-Pad2)
- K57 pad 1: Net-(K57-Pad1) -> Net-(K12-Pad1)
- K57 pad 2: Net-(K57-Pad2) -> Net-(D57-Pad2)
- K58 pad 1: Net-(K58-Pad1) -> Net-(K13-Pad1)
- K58 pad 2: Net-(K58-Pad2) -> Net-(D58-Pad2)
- K59 pad 1: Net-(K59-Pad1) -> Net-(K14-Pad1)
- K59 pad 2: Net-(K59-Pad2) -> Net-(D59-Pad2)
- K6 pad : Net-(U1-Pad16) -> (no net)
- K6 pad 1: Net-(K6-Pad1) -> Net-(K15-Pad1)
- K6 pad 2: Net-(K6-Pad2) -> Net-(D6-Pad2)
- K60 pad 1: Net-(K60-Pad1) -> Net-(K15-Pad1)
- K60 pad 2: Net-(K60-Pad2) -> Net-(D60-Pad2)
- K61 pad 1: Net-(K61-Pad1) -> Net-(K16-Pad1)
- K61 pad 2: Net-(K61-Pad2) -> Net-(D61-Pad2)
- K62 pad 1: Net-(K62-Pad1) -> Net-(K17-Pad1)
- K62 pad 2: Net-(K62-Pad2) -> Net-(D62-Pad2)
- K63 pad 1: Net-(K63-Pad1) -> Net-(K18-Pad1)
- K63 pad 2: Net-(K63-Pad2) -> Net-(D63-Pad2)
- K64 pad 1: Net-(K64-Pad1) -> Net-(K1-Pad1)
- K64 pad 2: Net-(K64-Pad2) -> Net-(D64-Pad2)
- K65 pad 1: Net-(K65-Pad1) -> Net-(K11-Pad1)
- K65 pad 2: Net-(K65-Pad2) -> Net-(D65-Pad2)
- K66 pad 1: Net-(K66-Pad1) -> Net-(K12-Pad1)
- K66 pad 2: Net-(K66-Pad2) -> Net-(D66-Pad2)
- K67 pad 1: Net-(K67-Pad1) -> Net-(K13-Pad1)
- K67 pad 2: Net-(K67-Pad2) -> Net-(D67-Pad2)
- K68 pad 1: Net-(K68-Pad1) -> Net-(K14-Pad1)
- K68 pad 2: Net-(K68-Pad2) -> Net-(D68-Pad2)
- K69 pad 1: Net-(K69-Pad1) -> Net-(K15-Pad1)
- K69 pad 2: Net-(K69-Pad2) -> Net-(D69-Pad2)
- K7 pad 1: Net-(K7-Pad1) -> Net-(K16-Pad1)
- K7 pad 2: Net-(K7-Pad2) -> Net-(D7-Pad2)
- K70 pad 1: Net-(K70-Pad1) -> Net-(K16-Pad1)
- K70 pad 2: Net-(K70-Pad2) -> Net-(D70-Pad2)
- K71 pad 1: Net-(K71-Pad1) -> Net-(K17-Pad1)
- K71 pad 2: Net-(K71-Pad2) -> Net-(D71-Pad2)
- K72 pad 1: Net-(K72-Pad1) -> Net-(K18-Pad1)
- K72 pad 2: Net-(K72-Pad2) -> Net-(D72-Pad2)
- K73 pad 1: Net-(K73-Pad1) -> Net-(K1-Pad1)
- K73 pad 2: Net-(K73-Pad2) -> Net-(D73-Pad2)
- K74 pad 1: Net-(K74-Pad1) -> Net-(K11-Pad1)
- K74 pad 2: Net-(K74-Pad2) -> Net-(D74-Pad2)
- K75 pad 1: Net-(K75-Pad1) -> Net-(K12-Pad1)
- K75 pad 2: Net-(K75-Pad2) -> Net-(D75-Pad2)
- K76 pad 1: Net-(K76-Pad1) -> Net-(K13-Pad1)
- K76 pad 2: Net-(K76-Pad2) -> Net-(D76-Pad2)
- K77 pad 1: Net-(K77-Pad1) -> Net-(K14-Pad1)
- K77 pad 2: Net-(K77-Pad2) -> Net-(D77-Pad2)
- K78 pad 1: Net-(K78-Pad1) -> Net-(K15-Pad1)
- K78 pad 2: Net-(K78-Pad2) -> Net-(D78-Pad2)
- K8 pad 1: Net-(K8-Pad1) -> Net-(K17-Pad1)
- K8 pad 2: Net-(K8-Pad2) -> Net-(D8-Pad2)
- K9 pad 1: Net-(K9-Pad1) -> Net-(K18-Pad1)
- K9 pad 2: Net-(K9-Pad2) -> Net-(D9-Pad2)
- U1 pad 12: Net-(U1-Pad12) -> Net-(K1-Pad1)
- U1 pad 13: Net-(U1-Pad13) -> Net-(K18-Pad1)
- U1 pad 14: Net-(U1-Pad14) -> Net-(K17-Pad1)
- U1 pad 15: Net-(U1-Pad15) -> Net-(K16-Pad1)
- U1 pad 16: Net-(U1-Pad16) -> Net-(K15-Pad1)
- U1 pad 17: Net-(U1-Pad17) -> Net-(K14-Pad1)
- U1 pad 18: Net-(U1-Pad18) -> Net-(K13-Pad1)
- U1 pad 19: Net-(U1-Pad19) -> Net-(K12-Pad1)
- U1 pad 20: Net-(U1-Pad20) -> Net-(K11-Pad1)
- U1 pad 21: Net-(U1-Pad21) -> (no net)
- U1 pad 22: Net-(U1-Pad22) -> Net-(SW1-Pad2)
- U1 pad 23: Net-(U1-Pad23) -> Net-(SW1-Pad1)
- U1 pad 24: Net-(U1-Pad24) -> (no net)
- U1 pad 3: Net-(U1-Pad3) -> (no net)
- U1 pad 4: Net-(U1-Pad4) -> (no net)
Routing:
- net (no net): track 1599.0 -> 0.00 mm
- net Net-(K18-Pad1): track 2.00 -> 581.7 mm, vias 0 -> 4
- net Net-(K17-Pad1): track 24.9 -> 579.8 mm, vias 0 -> 4
- net Net-(K15-Pad1): track 187.0 -> 622.8 mm, vias 0 -> 4
- net Net-(K73-Pad1): track 431.4 -> 0.00 mm
- net Net-(K11-Pad1): track 67.8 -> 436.3 mm, vias 0 -> 2
- net Net-(K12-Pad1): track 137.4 -> 390.7 mm, vias 0 -> 3
- net Net-(K13-Pad1): track 229.7 -> 448.2 mm, vias 0 -> 4
- net Net-(D46-Pad1): track 408.2 -> 625.6 mm, vias 0 -> 6
- net Net-(K16-Pad1): track 354.7 -> 563.8 mm, vias 0 -> 7
- net Net-(D73-Pad1): track 396.9 -> 585.6 mm, vias 0 -> 3
- net Net-(U1-Pad16): track 167.1 -> 0.00 mm
- net Net-(K14-Pad1): track 301.4 -> 465.8 mm, vias 0 -> 4
- net Net-(K65-Pad1): track 125.9 -> 0.00 mm
- net Net-(K1-Pad1): track 319.9 -> 444.6 mm, vias 0 -> 4
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Other:
- net class Default removed

Commit message: final
Parts:
- moved D67 37.7 mm to (309.1, 73.8)
- moved D1 37.7 mm to (18.6, 16.6)
- moved D11 37.7 mm to (209.1, 16.6)
- moved D12 37.7 mm to (228.1, 16.6)
- moved D13 37.7 mm to (247.2, 16.6)
- moved D14 37.7 mm to (266.2, 16.6)
- moved D15 37.7 mm to (294.8, 26.2)
- moved D16 37.7 mm to (304.3, 16.6)
- moved D17 37.7 mm to (323.4, 16.6)
- moved D18 37.7 mm to (352.0, 16.6)
- moved D2 37.7 mm to (37.6, 16.6)
- moved D3 37.7 mm to (56.7, 16.6)
- moved D33 37.7 mm to (294.8, 35.7)
- moved D36 37.7 mm to (354.3, 35.7)
- moved D4 37.7 mm to (75.7, 16.6)
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Routing:
- net Net-(D1-Pad1): track 120.7 -> 180.6 mm
- net Net-(D37-Pad1): track 208.0 -> 237.0 mm, vias 2 -> 4
- net Net-(D10-Pad1): track 321.7 -> 342.5 mm
Other:
- outline, holes or cut-outs redrawn
- rule pad_to_mask_clearance: 0.05 -> 0
